File: MC1201-ATX.kicad_sch (KiCad schematic)
At the start: 251 parts, among them J1 PLD-16, J2 PLD-16, J3 PLD-16, J4 ATX-20, J5 Conn_01x01_Pin, J6 Conn_01x01_Pin, J7 Conn_01x09_Pin, P1 Conn_01x01_Pin, P10 Conn_01x01_Pin, P11 Conn_01x01_Pin, P12 Conn_01x01_Pin, P13 Conn_01x01_Pin, P14 Conn_01x01_Pin, P15 Conn_01x01_Pin, P16 Conn_01x01_Pin, P17 Conn_01x01_Pin, P18 Conn_01x01_Pin, P2 Conn_01x01_Pin, P3 Conn_01x01_Pin, P4 Conn_01x01_Pin, P5 Conn_01x01_Pin, P6 Conn_01x01_Pin, P7 Conn_01x01_Pin, P8 Conn_01x01_Pin, P9 Conn_01x01_Pin, Q1 BC547, X2 AFPC, X3 QBUS_DWK_64Pin_MBT

Commit message: More updates.
Verified and documented incorrect Reset button connection (E0010). Debugged
address separator, removed extraneous RX5-CX1 delay.

The board boots up at this point.
Parts:
- CX1: now not fitted
- RX5: value 2K -> 0
Connections:
- net VCC: now also E12_9.2; no longer E12_9.1
- net RAM_RPLY renamed CSRAM
- net ~{RESET} renamed ~{INIT}
- net ~{INIT}: now also E12_9.1; no longer E12_9.2
Other:
- note added: "ERRATUM E0010 Неверное подключение кнопки Reset"
- note added: "Для этой платы дополнительная задержка ~{SYNC} не требуется"
- moved on the sheet: E12_1, E12_7, E4_1, E4_2, E4_3, E5_3, E5_6, E5_7, E5_8, E8_2, E8_3, E8_7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
