File: Fixes_Rev_0.1C/Fixes_Rev_0.1C.kicad_sch (KiCad schematic)
At the start: 9 parts, among them U1 1533LI1, U2 1533TM2, U3 1533LA8, U4 CD74HCT4067M, U5 1533LE4

Commit message: Fixes: Correct /INIT signal name, more comments.
Add more explanations on where to take some signals from. Name /INIT signal
correctly. Spotted by Pavel "Max232CPE".
Connections:
- net ~{RESET} renamed ~{INIT}
Other:
- note added: "Линии /INIT, /DOUT, /AD2, /AD3 подключить к системному разъему (X3)"
Changed lines of the file:
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@@
 		)
 	)
+	(text "Линии /INIT, /DOUT, /AD2, /AD3\nподключить к системному разъему (X3)"
+		(exclude_from_sim no)
+		(at 63.5 26.035 0)
+		(effects
+			(font
+				(size 1.27 1.27)
+			)
+			(justify right)
+		)
+	)
 	(junction
 		(at 71.12 179.07)
@@
 		)
 	)
-	(global_label "~{RESET}"
+	(global_label "~{INIT}"
 		(shape input)
 		(at 64.77 68.58 180)
@@
 		)
 		(property "Intersheetrefs" "${INTERSHEET_REFS}"
-			(at 56.0397 68.58 0)
+			(at 58.2771 68.58 0)
 			(hide yes)
 			(show_name no)
@@
 		)
 		(instances
-			(project "MemManager"
+			(project "Fixes_Rev_0.1C"
 				(path "/e8e5a0b4-44b9-4e84-b144-8989a57edfae"
 					(reference "U3")
@@
 		)
 		(instances
-			(project "MemManager"
+			(project "Fixes_Rev_0.1C"
 				(path "/e8e5a0b4-44b9-4e84-b144-8989a57edfae"
 					(reference "U3")
@@
 		)
 		(instances
-			(project "MemManager"
+			(project "Fixes_Rev_0.1C"
 				(path "/e8e5a0b4-44b9-4e84-b144-8989a57edfae"
 					(reference "D1")
@@
 		)
 		(instances
-			(project "MemManager"
+			(project "Fixes_Rev_0.1C"
 				(path "/e8e5a0b4-44b9-4e84-b144-8989a57edfae"
 					(reference "U3")
@@
 		)
 		(instances
-			(project "MemManager"
+			(project "Fixes_Rev_0.1C"
 				(path "/e8e5a0b4-44b9-4e84-b144-8989a57edfae"
 					(reference "U5")
@@
 		)
 		(instances
-			(project "MemManager"
+			(project "Fixes_Rev_0.1C"
 				(path "/e8e5a0b4-44b9-4e84-b144-8989a57edfae"
 					(reference "U5")
@@
 		)
 		(instances
-			(project "MemManager"
+			(project "Fixes_Rev_0.1C"
 				(path "/e8e5a0b4-44b9-4e84-b144-8989a57edfae"
 					(reference "U5")
@@
 		)
 		(instances
-			(project "MemManager"
+			(project "Fixes_Rev_0.1C"
 				(path "/e8e5a0b4-44b9-4e84-b144-8989a57edfae"
 					(reference "U5")
@@
 		)
 		(instances
-			(project "MemManager"
+			(project "Fixes_Rev_0.1C"
 				(path "/e8e5a0b4-44b9-4e84-b144-8989a57edfae"
 					(reference "U3")
@@
 		)
 		(instances
-			(project "MemManager"
+			(project "Fixes_Rev_0.1C"
 				(path "/e8e5a0b4-44b9-4e84-b144-8989a57edfae"
 					(reference "DD6")
@@
 		)
 		(instances
-			(project "MemManager"
+			(project "Fixes_Rev_0.1C"
 				(path "/e8e5a0b4-44b9-4e84-b144-8989a57edfae"
 					(reference "#PWR05")
@@
 		)
 		(instances
-			(project "MemManager"
+			(project "Fixes_Rev_0.1C"
 				(path "/e8e5a0b4-44b9-4e84-b144-8989a57edfae"
 					(reference "U4")
@@
 		)
 		(instances
-			(project "MemManager"
+			(project "Fixes_Rev_0.1C"
 				(path "/e8e5a0b4-44b9-4e84-b144-8989a57edfae"
 					(reference "R2")
@@
 		)
 		(instances
-			(project "MemManager"
+			(project "Fixes_Rev_0.1C"
 				(path "/e8e5a0b4-44b9-4e84-b144-8989a57edfae"
 					(reference "U3")
@@
 		)
 		(instances
-			(project "MemManager"
+			(project "Fixes_Rev_0.1C"
 				(path "/e8e5a0b4-44b9-4e84-b144-8989a57edfae"
 					(reference "R1")
@@
 		)
 		(instances
-			(project "MemManager"
+			(project "Fixes_Rev_0.1C"
 				(path "/e8e5a0b4-44b9-4e84-b144-8989a57edfae"
 					(reference "#PWR03")
@@
 		)
 		(instances
-			(project "MemManager"
+			(project "Fixes_Rev_0.1C"
 				(path "/e8e5a0b4-44b9-4e84-b144-8989a57edfae"
 					(reference "#PWR07")
@@
 		)
 		(instances
-			(project "MemManager"
+			(project "Fixes_Rev_0.1C"
 				(path "/e8e5a0b4-44b9-4e84-b144-8989a57edfae"
 					(reference "#PWR01")
@@
 		)
 		(instances
-			(project "MemManager"
+			(project "Fixes_Rev_0.1C"
 				(path "/e8e5a0b4-44b9-4e84-b144-8989a57edfae"
 					(reference "U1")
@@
 		)
 		(instances
-			(project "MemManager"
+			(project "Fixes_Rev_0.1C"
 				(path "/e8e5a0b4-44b9-4e84-b144-8989a57edfae"
 					(reference "U1")
@@
 		)
 		(instances
-			(project "MemManager"
+			(project "Fixes_Rev_0.1C"
 				(path "/e8e5a0b4-44b9-4e84-b144-8989a57edfae"
 					(reference "U1")
@@
 		)
 		(instances
-			(project "MemManager"
+			(project "Fixes_Rev_0.1C"
 				(path "/e8e5a0b4-44b9-4e84-b144-8989a57edfae"
 					(reference "U1")
@@
 		)
 		(instances
-			(project "MemManager"
+			(project "Fixes_Rev_0.1C"
 				(path "/e8e5a0b4-44b9-4e84-b144-8989a57edfae"
 					(reference "U1")
@@
 		)
 		(instances
-			(project "MemManager"
+			(project "Fixes_Rev_0.1C"
 				(path "/e8e5a0b4-44b9-4e84-b144-8989a57edfae"
 					(reference "#PWR02")
@@
 		)
 		(instances
-			(project "MemManager"
+			(project "Fixes_Rev_0.1C"
 				(path "/e8e5a0b4-44b9-4e84-b144-8989a57edfae"
 					(reference "DD6")
@@
 		)
 		(instances
-			(project "MemManager"
+			(project "Fixes_Rev_0.1C"
 				(path "/e8e5a0b4-44b9-4e84-b144-8989a57edfae"
 					(reference "U2")
@@
 		)
 		(instances
-			(project "MemManager"
+			(project "Fixes_Rev_0.1C"
 				(path "/e8e5a0b4-44b9-4e84-b144-8989a57edfae"
 					(reference "U2")
@@
 		)
 		(instances
-			(project "MemManager"
+			(project "Fixes_Rev_0.1C"
 				(path "/e8e5a0b4-44b9-4e84-b144-8989a57edfae"
 					(reference "U2")
@@
 		)
 		(instances
-			(project "MemManager"
+			(project "Fixes_Rev_0.1C"
 				(path "/e8e5a0b4-44b9-4e84-b144-8989a57edfae"
 					(reference "#PWR04")
@@
 		)
 		(instances
-			(project "MemManager"
+			(project "Fixes_Rev_0.1C"
 				(path "/e8e5a0b4-44b9-4e84-b144-8989a57edfae"
 					(reference "#PWR06")
