File: Motherboard_Rev_0.1C/MC1201-ATX.kicad_sch (KiCad schematic)
At the start: 251 parts, among them J1 PLD-16, J2 PLD-16, J3 PLD-16, J4 ATX-20, J5 Conn_01x01_Pin, J6 Conn_01x01_Pin, J7 Conn_01x09_Pin, P1 Conn_01x01_Pin, P10 Conn_01x01_Pin, P11 Conn_01x01_Pin, P12 Conn_01x01_Pin, P13 Conn_01x01_Pin, P14 Conn_01x01_Pin, P15 Conn_01x01_Pin, P16 Conn_01x01_Pin, P17 Conn_01x01_Pin, P18 Conn_01x01_Pin, P2 Conn_01x01_Pin, P3 Conn_01x01_Pin, P4 Conn_01x01_Pin, P5 Conn_01x01_Pin, P6 Conn_01x01_Pin, P7 Conn_01x01_Pin, P8 Conn_01x01_Pin, P9 Conn_01x01_Pin, Q1 BC547, X2 AFPC, X3 QBUS_DWK_64Pin_MBT

Commit message: Update state of the build
Built and tested the mezzanine board. Brought README up to date, corrected
links.
Parts:
- removed P2, P4: Conn_01x01_Pin, Connector_PinHeader_2.54mm:PinHeader_1x01_P2.54mm_Vertical, symbol Connector:Conn_01x01_Pin
- E5_4: now fitted
Connections:
- net LOCK is gone; now on an unnamed net: DD5.5, DD9.9
- net ~{DOUT}: now also DD6.9
- net ~{RPLY}: no longer DD8.2 (D), E5_4.2
- net at DD17.10 (~{S}), DD18.10 (~{S}), DD18.13 (~{R})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: now also DD44.13 (~{R})
- net SEL1: now reaches DD10.11, DD6.4
- net DOUT: now reaches DD6.8, P3.1 (Pin_1)
- net ~{CPU_DOUT}: now reaches DD5.3, DD7.37 (DOUT), E4_4.2
- net ~{CPU_DIN}: now reaches DD6.1, DD7.38 (DIN), E5_2.2
- net ~{LOCK}: now reaches DD6.13, P1.1 (Pin_1)
- net SYSMEM renamed SYSRAM
- new net ~{CPU_RPLY}: DD8.2 (D), E5_4.2
- no-connect marks 35 -> 34
Other:
- note added: "ERRATUM E0003. Цепь ~{RPLY} соединяется через буфер на мезонинной плате"
- note added: "ERRATUM E0005 Сформировать сигнал LOCK с помощью свободного инвертора DD6F."
- note added: "J1 и J2: устанавливать разъемы 7x2. Позиции 1-2 не задействовать"
- note added: "Вместо DX3 и DX4 установить разъёмы для подключения мезонинной платы"
- note added: "К разъему J8 мезонинной платы"
- note added: "Сформировать сигнал DOUT с помощью свободного инвертора DD6D"
- note removed: "ERRATUM E0003 ~{RPLY} не подключен."
- note removed: "ERRATUM E0005 Сигнал LOCK не реализован."
- note removed: "ERRATUM E0008 Не декодируется окно системного ОЗУ 177600_{8}..177677_{8}"
- moved on the sheet: DD6D, DD6F, P1, P3
