File: QBus_MPISlots/QBus.kicad_sch (KiCad schematic)
At the start: 5 parts, among them J1 QBUSDUAL, J2 QBUSDUAL, J3 QBUSDUAL, J4 QBUSDUAL, J5 IDC-64M

Commit message: QBus_MPISlots: Add 12V connectors
12V voltages aren't present on the main connector. Use auxiliary ATX connector
for +12V and extra pins for -12V.
Parts:
- added J6: Conn_02x02_Top_Bottom, Connector_Molex:Molex_Mini-Fit_Jr_5566-04A_2x02_P4.20mm_Vertical, symbol Connector_Generic:Conn_02x02_Top_Bottom
- added J7: Conn_01x03, Connector_Wago:Wago_734-133_1x03_P3.50mm_Vertical, symbol Connector_Generic:Conn_01x03
Connections:
- net +12V: now also J6.1 (Pin_1), J6.2 (Pin_2), J7.1 (Pin_1)
- net -12V: now also J7.2 (Pin_2)
- net GND: now also J6.3 (Pin_3), J6.4 (Pin_4), J7.3 (Pin_3)
